Commit message: leader_follower robot

File: description/urdf/supre_robot.urdf.xacro (robot description, xacro)
@@ -14,6 +14,7 @@
   <!-- Import gripper description -->
   <xacro:include filename="$(find supre_robot_control)/ros2_control/gripper.ros2_control.xacro" />
-  <xacro:supre_robot>
-  </xacro:supre_robot>
+  <link name="world"/>
+  <xacro:create_robot>
+  </xacro:create_robot>
   <xacro:gripper_system
     name="MisumiGripper" prefix="$(arg prefix)"

File: description/urdf/supre_robot_description.urdf.xacro (robot description, xacro)
@@ -1,13 +1,12 @@
 <?xml version="1.0"?>
-<robot xmlns:xacro="http://www.ros.org/wiki/xacro">
-  <xacro:macro name="supre_robot">
+<robot xmlns:xacro="http://www.ros.org/wiki/xacro" params="name prefix">
+  <xacro:macro name="create_robot">
     <!-- Used for fixing robot to Gazebo 'world' -->
-    <link name="world"/>
-    <joint name="base_joint" type="fixed">
+    <joint name="${prefix}base_joint" type="fixed">
         <parent link="world"/>
-        <child link="base_link"/>
+        <child link="${prefix}base_link"/>
         <origin xyz="0 0 0" rpy="0 0 0"/>
     </joint>
-    <link name="base_link">
+    <link name="${prefix}base_link">
         <visual>
             <geometry>
@@ -24,5 +23,5 @@
         </collision>
     </link>
-    <link name="gripper_finger_link">
+    <link name="${prefix}gripper_finger_link">
         <visual>
             <geometry>
@@ -40,7 +39,7 @@
         </inertial>
     </link>
-    <joint name="gripper_joint" type="prismatic">
-        <parent link="base_link"/>
-        <child link="gripper_finger_link"/>
+    <joint name="${prefix}gripper_joint" type="prismatic">
+        <parent link="${prefix}base_link"/>
+        <child link="${prefix}gripper_finger_link"/>
         <origin xyz="0 0 0" rpy="0 0 0"/>
         <axis xyz="1 0 0"/>
