Commit message: fix

File: description/urdf/supre_robot_description.urdf.xacro (robot description, xacro)
@@ -1,5 +1,5 @@
 <?xml version="1.0"?>
-<robot xmlns:xacro="http://www.ros.org/wiki/xacro" params="name prefix">
-  <xacro:macro name="create_robot">
+<robot xmlns:xacro="http://www.ros.org/wiki/xacro">
+  <xacro:macro name="create_robot" params="name prefix">
     <!-- Used for fixing robot to Gazebo 'world' -->
     <joint name="${prefix}base_joint" type="fixed">

Commit message: fix

File: description/urdf/supre_robot_description.urdf.xacro (robot description, xacro)
@@ -1,5 +1,5 @@
 <?xml version="1.0"?>
 <robot xmlns:xacro="http://www.ros.org/wiki/xacro">
-  <xacro:macro name="create_robot" params="name prefix">
+  <xacro:macro name="create_robot" params="prefix">
     <!-- Used for fixing robot to Gazebo 'world' -->
     <joint name="${prefix}base_joint" type="fixed">
