Commit message: leader follower

File: description/urdf/leader_supre_robot_description.urdf.xacro (robot description, xacro)
@@ -23,20 +23,4 @@
         </collision>
     </link>
-    <link name="${prefix}gripper_finger_link">
-        <visual>
-            <geometry>
-                <box size="0.1 0.02 0.02"/>
-            </geometry>
-        </visual>
-        <collision>
-            <geometry>
-                <box size="0.1 0.02 0.02"/>
-            </geometry>
-        </collision>
-        <inertial>
-            <mass value="0.1"/>
-            <inertia ixx="0.001" ixy="0" ixz="0" iyy="0.001" iyz="0" izz="0.001"/>
-        </inertial>
-    </link>
   </xacro:macro>
 </robot>
