Commit message: leader follower

File: description/ros2_control/leader_joints.ros2_control.xacro (robot description, xacro)
@@ -13,5 +13,5 @@
         <joint name="${prefix}left_arm_joint_1">
             <param name="node_id">21</param>
-            <param name="start_enabled">true</param>
+            <param name="start_enabled">false</param>
             <command_interface name="position"/>
             <state_interface name="position"/>
@@ -20,5 +20,5 @@
         <joint name="${prefix}left_arm_joint_2">
             <param name="node_id">22</param>
-            <param name="start_enabled">true</param>
+            <param name="start_enabled">false</param>
             <command_interface name="position"/>
             <state_interface name="position"/>
@@ -27,5 +27,5 @@
         <joint name="${prefix}left_arm_joint_3">
             <param name="node_id">23</param>
-            <param name="start_enabled">true</param>
+            <param name="start_enabled">false</param>
             <command_interface name="position"/>
             <state_interface name="position"/>
@@ -34,5 +34,5 @@
         <joint name="${prefix}left_arm_joint_4">
             <param name="node_id">24</param>
-            <param name="start_enabled">true</param>
+            <param name="start_enabled">false</param>
             <command_interface name="position"/>
             <state_interface name="position"/>
@@ -41,5 +41,5 @@
         <joint name="${prefix}left_arm_joint_5">
             <param name="node_id">25</param>
-            <param name="start_enabled">true</param>
+            <param name="start_enabled">false</param>
             <command_interface name="position"/>
             <state_interface name="position"/>
@@ -48,5 +48,12 @@
         <joint name="${prefix}left_arm_joint_6">
             <param name="node_id">26</param>
-            <param name="start_enabled">true</param>
+            <param name="start_enabled">false</param>
+            <command_interface name="position"/>
+            <state_interface name="position"/>
+            <state_interface name="velocity"/>
+        </joint>
+        <joint name="${prefix}left_arm_joint_7">
+            <param name="node_id">27</param>
+            <param name="start_enabled">false</param>
             <command_interface name="position"/>
             <state_interface name="position"/>
@@ -56,5 +63,5 @@
         <joint name="${prefix}right_arm_joint_1">
             <param name="node_id">11</param>
-            <param name="start_enabled">true</param>
+            <param name="start_enabled">false</param>
             <command_interface name="position"/>
             <state_interface name="position"/>
@@ -63,5 +70,5 @@
         <joint name="${prefix}right_arm_joint_2">
             <param name="node_id">12</param>
-            <param name="start_enabled">true</param>
+            <param name="start_enabled">false</param>
             <command_interface name="position"/>
             <state_interface name="position"/>
@@ -70,5 +77,4 @@
         <joint name="${prefix}right_arm_joint_3">
             <param name="node_id">13</param>
-            <param name="start_enabled">true</param>
             <command_interface name="position"/>
             <state_interface name="position"/>
@@ -77,5 +83,5 @@
         <joint name="${prefix}right_arm_joint_4">
             <param name="node_id">14</param>
-            <param name="start_enabled">true</param>
+            <param name="start_enabled">false</param>
             <command_interface name="position"/>
             <state_interface name="position"/>
@@ -84,5 +90,5 @@
         <joint name="${prefix}right_arm_joint_5">
             <param name="node_id">15</param>
-            <param name="start_enabled">true</param>
+            <param name="start_enabled">false</param>
             <command_interface name="position"/>
             <state_interface name="position"/>
@@ -91,5 +97,11 @@
         <joint name="${prefix}right_arm_joint_6">
             <param name="node_id">16</param>
-            <param name="start_enabled">true</param>
+            <command_interface name="position"/>
+            <state_interface name="position"/>
+            <state_interface name="velocity"/>
+        </joint>
+        <joint name="${prefix}right_arm_joint_7">
+            <param name="node_id">17</param>
+            <param name="start_enabled">false</param>
             <command_interface name="position"/>
             <state_interface name="position"/>

File: description/urdf/follower_supre_robot.urdf.xacro (robot description, xacro)
@@ -3,5 +3,5 @@
   <xacro:arg name="use_mock_hardware" default="false" />
   <xacro:arg name="prefix" default="" />
-  <xacro:arg name="param_can_device_index" default="0" />
+  <xacro:arg name="param_can_device_index" default="1" />
   <xacro:arg name="param_can_baud_rate" default="1000" />
   <xacro:arg name="param_device" default="/dev/ttyTHS1" />
@@ -17,4 +17,5 @@
   <xacro:create_robot prefix="$(arg prefix)">
   </xacro:create_robot>
+<!--
   <xacro:gripper_system
     name="FollowerMisumiGripper" prefix="$(arg prefix)"
@@ -24,4 +25,5 @@
     param_baud_rate="$(arg param_baud_rate)"
     param_max_stroke="$(arg param_max_stroke)" />
+-->
   <xacro:joints_system
     name="FollowerEyouSystem" prefix="$(arg prefix)"

File: description/urdf/leader_supre_robot.urdf.xacro (robot description, xacro)
@@ -11,5 +11,5 @@
   <xacro:include filename="$(find supre_robot_control)/urdf/leader_supre_robot_description.urdf.xacro" />
   <!-- Import joints ros2_control description -->
-  <xacro:include filename="$(find supre_robot_control)/ros2_control/joints.ros2_control.xacro" />
+  <xacro:include filename="$(find supre_robot_control)/ros2_control/leader_joints.ros2_control.xacro" />
   <link name="world"/>
   <xacro:create_robot prefix="$(arg prefix)">

Commit message: leader follower

File: description/ros2_control/leader_joints.ros2_control.xacro (robot description, xacro)
@@ -53,11 +53,4 @@
             <state_interface name="velocity"/>
         </joint>
-        <joint name="${prefix}left_arm_joint_7">
-            <param name="node_id">27</param>
-            <param name="start_enabled">false</param>
-            <command_interface name="position"/>
-            <state_interface name="position"/>
-            <state_interface name="velocity"/>
-        </joint>
         <!-- Right Arm Joints -->
         <joint name="${prefix}right_arm_joint_1">
@@ -101,11 +94,4 @@
             <state_interface name="velocity"/>
         </joint>
-        <joint name="${prefix}right_arm_joint_7">
-            <param name="node_id">17</param>
-            <param name="start_enabled">false</param>
-            <command_interface name="position"/>
-            <state_interface name="position"/>
-            <state_interface name="velocity"/>
-        </joint>
     </ros2_control>
   </xacro:macro>

Commit message: gripper

File: description/ros2_control/leader_joints.ros2_control.xacro (robot description, xacro)
@@ -96,4 +96,10 @@
             <state_interface name="velocity"/>
         </joint>
+        <joint name="${prefix}right_arm_joint_7">
+            <param name="node_id">17</param>
+            <command_interface name="position"/>
+            <state_interface name="position"/>
+            <state_interface name="velocity"/>
+        </joint>
     </ros2_control>
   </xacro:macro>

File: description/urdf/follower_supre_robot.urdf.xacro (robot description, xacro)
@@ -17,5 +17,4 @@
   <xacro:create_robot prefix="$(arg prefix)">
   </xacro:create_robot>
-<!--
   <xacro:gripper_system
     name="FollowerMisumiGripper" prefix="$(arg prefix)"
@@ -25,5 +24,4 @@
     param_baud_rate="$(arg param_baud_rate)"
     param_max_stroke="$(arg param_max_stroke)" />
--->
   <xacro:joints_system
     name="FollowerEyouSystem" prefix="$(arg prefix)"

Commit message: test

File: description/ros2_control/leader_joints.ros2_control.xacro (robot description, xacro)
@@ -47,4 +47,11 @@
         </joint>
         <joint name="${prefix}left_arm_joint_6">
+            <param name="node_id">26</param>
+            <param name="start_enabled">false</param>
+            <command_interface name="position"/>
+            <state_interface name="position"/>
+            <state_interface name="velocity"/>
+        </joint>
+        <joint name="${prefix}left_arm_joint_7">
             <param name="node_id">26</param>
             <param name="start_enabled">false</param>
