Commit message: remove gripper from common

File: description/ros2_control/gripper_follower_joints.ros2_control copy.xacro (robot description, xacro)
@@ -12,6 +12,6 @@
         <!-- Left Arm Joints -->
         <joint name="${prefix}left_arm_joint_1">
-            <param name="node_id">22</param>
-            <param name="start_enabled">false</param>
+            <param name="node_id">21</param>
+            <param name="start_enabled">true</param>
             <command_interface name="position"/>
             <state_interface name="position"/>
@@ -19,6 +19,6 @@
         </joint>
         <joint name="${prefix}left_arm_joint_2">
-            <param name="node_id">21</param>
-            <param name="start_enabled">false</param>
+            <param name="node_id">22</param>
+            <param name="start_enabled">true</param>
             <command_interface name="position"/>
             <state_interface name="position"/>
@@ -27,5 +27,5 @@
         <joint name="${prefix}left_arm_joint_3">
             <param name="node_id">23</param>
-            <param name="start_enabled">false</param>
+            <param name="start_enabled">true</param>
             <command_interface name="position"/>
             <state_interface name="position"/>
@@ -34,5 +34,5 @@
         <joint name="${prefix}left_arm_joint_4">
             <param name="node_id">24</param>
-            <param name="start_enabled">false</param>
+            <param name="start_enabled">true</param>
             <command_interface name="position"/>
             <state_interface name="position"/>
@@ -41,5 +41,5 @@
         <joint name="${prefix}left_arm_joint_5">
             <param name="node_id">25</param>
-            <param name="start_enabled">false</param>
+            <param name="start_enabled">true</param>
             <command_interface name="position"/>
             <state_interface name="position"/>
@@ -48,5 +48,5 @@
         <joint name="${prefix}left_arm_joint_6">
             <param name="node_id">26</param>
-            <param name="start_enabled">false</param>
+            <param name="start_enabled">true</param>
             <command_interface name="position"/>
             <state_interface name="position"/>
@@ -55,6 +55,6 @@
         <!-- Right Arm Joints -->
         <joint name="${prefix}right_arm_joint_1">
-            <param name="node_id">12</param>
-            <param name="start_enabled">false</param>
+            <param name="node_id">11</param>
+            <param name="start_enabled">true</param>
             <command_interface name="position"/>
             <state_interface name="position"/>
@@ -62,6 +62,6 @@
         </joint>
         <joint name="${prefix}right_arm_joint_2">
-            <param name="node_id">11</param>
-            <param name="start_enabled">false</param>
+            <param name="node_id">12</param>
+            <param name="start_enabled">true</param>
             <command_interface name="position"/>
             <state_interface name="position"/>
@@ -70,5 +70,5 @@
         <joint name="${prefix}right_arm_joint_3">
             <param name="node_id">13</param>
-            <param name="start_enabled">false</param>
+            <param name="start_enabled">true</param>
             <command_interface name="position"/>
             <state_interface name="position"/>
@@ -77,5 +77,5 @@
         <joint name="${prefix}right_arm_joint_4">
             <param name="node_id">14</param>
-            <param name="start_enabled">false</param>
+            <param name="start_enabled">true</param>
             <command_interface name="position"/>
             <state_interface name="position"/>
@@ -84,5 +84,5 @@
         <joint name="${prefix}right_arm_joint_5">
             <param name="node_id">15</param>
-            <param name="start_enabled">false</param>
+            <param name="start_enabled">true</param>
             <command_interface name="position"/>
             <state_interface name="position"/>
@@ -91,5 +91,5 @@
         <joint name="${prefix}right_arm_joint_6">
             <param name="node_id">16</param>
-            <param name="start_enabled">false</param>
+            <param name="start_enabled">true</param>
             <command_interface name="position"/>
             <state_interface name="position"/>

File: description/ros2_control/gripper_leader_joints.ros2_control copy.xacro (robot description, xacro)
@@ -96,4 +96,11 @@
             <state_interface name="velocity"/>
         </joint>
+        <joint name="${prefix}right_arm_joint_7">
+            <param name="node_id">17</param>
+            <param name="start_enabled">false</param>
+            <command_interface name="position"/>
+            <state_interface name="position"/>
+            <state_interface name="velocity"/>
+        </joint>
     </ros2_control>
   </xacro:macro>

File: description/urdf/gripper_follower_supre_robot.urdf.xacro (robot description, xacro)
@@ -16,4 +16,10 @@
   <xacro:create_robot prefix="$(arg prefix)">
   </xacro:create_robot>
+  <xacro:gripper_system
+    name="FollowerMisumiGripper" prefix="$(arg prefix)"
+    use_mock_hardware="$(arg use_mock_hardware)"
+    param_device="$(arg param_device)"
+    param_baud_rate="$(arg param_baud_rate)"
+    param_max_stroke="$(arg param_max_stroke)" />
   <xacro:joints_system
     name="FollowerEyouSystem" prefix="$(arg prefix)"
