Commit message: launch

File: description/ros2_control/gripper.ros2_control.xacro (robot description, xacro)
@@ -15,8 +15,8 @@
             <command_interface name="position">
                 <param name="min">0</param>
-                <param name="max">${param}</param>
+                <param name="max">${param_max_stroke}</param>
             </command_interface>
             <state_interface name="position"/>
         </joint>
     </ros2_control>
-  </xacro:macro>
+</xacro:macro>

File: description/urdf/supre_robot.urdf.xacro (robot description, xacro)
@@ -1,3 +1,3 @@
-<robot xmlns:xacro="http://www.ros.org/wiki/xacro" name="2dof_robot">
+<robot xmlns:xacro="http://www.ros.org/wiki/xacro" name="supre_robot">
   <!-- Enable setting arguments from the launch file -->
   <xacro:arg name="use_mock_hardware" default="false" />
@@ -10,7 +10,7 @@
   <xacro:arg name="param_max_stroke" default=0.04 />
   <!-- Import joints ros2_control description -->
-  <xacro:include filename="$(find supre_robot_control)/description/ros2_control/joints.ros2_control.xacro" />
+  <xacro:include filename="$(find supre_robot_control)/ros2_control/joints.ros2_control.xacro" />
   <!-- Import gripper description -->
-  <xacro:include filename="$(find supre_robot_control)/description/ros2_control/gripper.ros2_control.xacro" />
+  <xacro:include filename="$(find supre_robot_control)/ros2_control/gripper.ros2_control.xacro" />
   <xacro:gripper_system
     name="MisumiGripper" prefix="$(arg prefix)"

Commit message: add namespace and prefix to adapt leader/follower robot arms

File: description/ros2_control/gripper.ros2_control.xacro (robot description, xacro)
@@ -13,5 +13,5 @@
         <!-- Define the single joint for the gripper -->
         <!-- The max_stroke should match your gripper's physical maximum opening in meters -->
-        <joint name="gripper_joint">
+        <joint name="${prefix}gripper_joint">
             <command_interface name="position">
                 <param name="min">0</param>

File: description/ros2_control/joints.ros2_control.xacro (robot description, xacro)
@@ -11,5 +11,5 @@
         </hardware>
         <!-- Left Arm Joints -->
-        <joint name="left_arm_joint_1">
+        <joint name="${prefix}left_arm_joint_1">
             <param name="node_id">21</param>
             <param name="start_enabled">false</param>
@@ -18,5 +18,5 @@
             <state_interface name="velocity"/>
         </joint>
-        <joint name="left_arm_joint_2">
+        <joint name="${prefix}left_arm_joint_2">
             <param name="node_id">22</param>
             <param name="start_enabled">false</param>
@@ -25,5 +25,5 @@
             <state_interface name="velocity"/>
         </joint>
-        <joint name="left_arm_joint_3">
+        <joint name="${prefix}left_arm_joint_3">
             <param name="node_id">23</param>
             <param name="start_enabled">false</param>
@@ -32,5 +32,5 @@
             <state_interface name="velocity"/>
         </joint>
-        <joint name="left_arm_joint_4">
+        <joint name="${prefix}left_arm_joint_4">
             <param name="node_id">24</param>
             <param name="start_enabled">false</param>
@@ -39,5 +39,5 @@
             <state_interface name="velocity"/>
         </joint>
-        <joint name="left_arm_joint_5">
+        <joint name="${prefix}left_arm_joint_5">
             <param name="node_id">25</param>
             <param name="start_enabled">false</param>
@@ -46,5 +46,5 @@
             <state_interface name="velocity"/>
         </joint>
-        <joint name="left_arm_joint_6">
+        <joint name="${prefix}left_arm_joint_6">
             <param name="node_id">26</param>
             <param name="start_enabled">false</param>
@@ -53,5 +53,5 @@
             <state_interface name="velocity"/>
         </joint>
-        <joint name="left_arm_joint_7">
+        <joint name="${prefix}left_arm_joint_7">
             <param name="node_id">27</param>
             <param name="start_enabled">false</param>
@@ -61,5 +61,5 @@
         </joint>
         <!-- Right Arm Joints -->
-        <joint name="right_arm_joint_1">
+        <joint name="${prefix}right_arm_joint_1">
             <param name="node_id">11</param>
             <command_interface name="position"/>
@@ -67,5 +67,5 @@
             <state_interface name="velocity"/>
         </joint>
-        <joint name="right_arm_joint_2">
+        <joint name="${prefix}right_arm_joint_2">
             <param name="node_id">12</param>
             <command_interface name="position"/>
@@ -73,5 +73,5 @@
             <state_interface name="velocity"/>
         </joint>
-        <joint name="right_arm_joint_3">
+        <joint name="${prefix}right_arm_joint_3">
             <param name="node_id">13</param>
             <command_interface name="position"/>
@@ -79,5 +79,5 @@
             <state_interface name="velocity"/>
         </joint>
-        <joint name="right_arm_joint_4">
+        <joint name="${prefix}right_arm_joint_4">
             <param name="node_id">14</param>
             <command_interface name="position"/>
@@ -85,5 +85,5 @@
             <state_interface name="velocity"/>
         </joint>
-        <joint name="right_arm_joint_5">
+        <joint name="${prefix}right_arm_joint_5">
             <param name="node_id">15</param>
             <command_interface name="position"/>
@@ -91,5 +91,5 @@
             <state_interface name="velocity"/>
         </joint>
-        <joint name="right_arm_joint_6">
+        <joint name="${prefix}right_arm_joint_6">
             <param name="node_id">16</param>
             <command_interface name="position"/>
@@ -97,5 +97,5 @@
             <state_interface name="velocity"/>
         </joint>
-        <joint name="right_arm_joint_7">
+        <joint name="${prefix}right_arm_joint_7">
             <param name="node_id">17</param>
             <command_interface name="position"/>

File: description/urdf/supre_robot.urdf.xacro (robot description, xacro)
@@ -17,5 +17,5 @@
   </xacro:supre_robot>
   <xacro:gripper_system
-    name="MisumiGripper" prefix="$(arg prefix)"
+    name="MisumiGripper" prefix="leader_"
     use_mock_hardware="$(arg use_mock_hardware)"
     param_device="$(arg param_device)"
@@ -24,5 +24,5 @@
     param_max_stroke="$(arg param_max_stroke)" />
   <xacro:joints_system
-    name="EyouSystem" prefix="$(arg prefix)"
+    name="EyouSystem" prefix="leader_"
     use_mock_hardware="$(arg use_mock_hardware)"
     param_can_device_index="$(arg param_can_device_index)"

Commit message: leader_follower

File: description/ros2_control/gripper.ros2_control.xacro (robot description, xacro)
@@ -13,5 +13,12 @@
         <!-- Define the single joint for the gripper -->
         <!-- The max_stroke should match your gripper's physical maximum opening in meters -->
-        <joint name="${prefix}gripper_joint">
+        <joint name="${prefix}left_arm_joint_7">
+            <command_interface name="position">
+                <param name="min">0</param>
+                <param name="max">${param_max_stroke}</param>
+            </command_interface>
+            <state_interface name="position"/>
+        </joint>
+        <joint name="${prefix}right_arm_joint_7">
             <command_interface name="position">
                 <param name="min">0</param>

File: description/urdf/follower_supre_robot.urdf.xacro (robot description, xacro)
@@ -9,12 +9,21 @@
   <xacro:arg name="param_baud_rate" default="115200" />
   <xacro:arg name="param_max_stroke" default="0.04" />
-  <xacro:include filename="$(find supre_robot_control)/urdf/leader_supre_robot_description.urdf.xacro" />
+  <xacro:include filename="$(find supre_robot_control)/urdf/supre_robot_description.urdf.xacro" />
   <!-- Import joints ros2_control description -->
-  <xacro:include filename="$(find supre_robot_control)/ros2_control/joints.ros2_control.xacro" />
+  <xacro:include filename="$(find supre_robot_control)/ros2_control/follower_joints.ros2_control.xacro" />
+  <!-- Import gripper description -->
+  <xacro:include filename="$(find supre_robot_control)/ros2_control/gripper.ros2_control.xacro" />
   <link name="world"/>
   <xacro:create_robot prefix="$(arg prefix)">
   </xacro:create_robot>
+  <xacro:gripper_system
+    name="FollowerMisumiGripper" prefix="$(arg prefix)"
+    use_mock_hardware="$(arg use_mock_hardware)"
+    param_device="$(arg param_device)"
+    param_slave_id="$(arg param_slave_id)"
+    param_baud_rate="$(arg param_baud_rate)"
+    param_max_stroke="$(arg param_max_stroke)" />
   <xacro:joints_system
-    name="LeaderEyouSystem" prefix="$(arg prefix)"
+    name="FollowerEyouSystem" prefix="$(arg prefix)"
     use_mock_hardware="$(arg use_mock_hardware)"
     param_can_device_index="$(arg param_can_device_index)"

Commit message: gripper

File: description/ros2_control/gripper.ros2_control.xacro (robot description, xacro)
@@ -13,15 +13,9 @@
         <!-- Define the single joint for the gripper -->
         <!-- The max_stroke should match your gripper's physical maximum opening in meters -->
-        <joint name="${prefix}left_arm_joint_7">
-            <command_interface name="position">
-                <param name="min">0</param>
-                <param name="max">${param_max_stroke}</param>
-            </command_interface>
-            <state_interface name="position"/>
-        </joint>
         <joint name="${prefix}right_arm_joint_7">
             <command_interface name="position">
                 <param name="min">0</param>
                 <param name="max">${param_max_stroke}</param>
+                <param name="slave_id">17</param>
             </command_interface>
             <state_interface name="position"/>

File: description/ros2_control/leader_joints.ros2_control.xacro (robot description, xacro)
@@ -53,11 +53,4 @@
             <state_interface name="velocity"/>
         </joint>
-        <joint name="${prefix}left_arm_joint_7">
-            <param name="node_id">26</param>
-            <param name="start_enabled">false</param>
-            <command_interface name="position"/>
-            <state_interface name="position"/>
-            <state_interface name="velocity"/>
-        </joint>
         <!-- Right Arm Joints -->
         <joint name="${prefix}right_arm_joint_1">
@@ -105,4 +98,5 @@
         <joint name="${prefix}right_arm_joint_7">
             <param name="node_id">17</param>
+            <param name="start_enabled">false</param>
             <command_interface name="position"/>
             <state_interface name="position"/>

Commit message: test

File: description/ros2_control/gripper.ros2_control.xacro (robot description, xacro)
@@ -1,10 +1,9 @@
 <?xml version="1.0"?>
 <robot xmlns:xacro="http://www.ros.org/wiki/xacro">
-<xacro:macro name="gripper_system" params="name prefix use_mock_hardware:=^|true param_device:=/dev/ttyTHS1 param_slave_id:=10 param_baud_rate:=115200 param_max_stroke:=0.04">
+<xacro:macro name="gripper_system" params="name prefix use_mock_hardware:=^|true param_device:=/dev/ttyTHS1  param_baud_rate:=115200 param_max_stroke:=0.04">
     <ros2_control name="${name}" type="system">
         <hardware>
           <plugin>supre_robot_control/MisumiGripperHardware</plugin>
           <param name="device">${param_device}</param>
-          <param name="slave_id">${param_slave_id}</param>
           <param name="baud_rate">${param_baud_rate}</param>
           <param name="default_speed_percent">100</param>

Commit message: jodell

File: description/ros2_control/gripper.ros2_control.xacro (robot description, xacro)
@@ -4,5 +4,5 @@
     <ros2_control name="${name}" type="system">
         <hardware>
-          <plugin>supre_robot_control/MisumiGripperHardware</plugin>
+          <plugin>supre_robot_control/JodellGripperHardware</plugin>
           <param name="device">${param_device}</param>
           <param name="baud_rate">${param_baud_rate}</param>
@@ -12,5 +12,5 @@
         <!-- Define the single joint for the gripper -->
         <!-- The max_stroke should match your gripper's physical maximum opening in meters -->
-        <joint name="${prefix}right_arm_joint_7">
+        <joint name="${prefix}left_arm_joint_7">
             <command_interface name="position">
                 <param name="min">0</param>
@@ -18,5 +18,5 @@
             </command_interface>
             <state_interface name="position"/>
-            <param name="slave_id">17</param>
+            <param name="slave_id">27</param>
         </joint>
     </ros2_control>

File: description/ros2_control/gripper_leader_joints.ros2_control.xacro (robot description, xacro)
@@ -53,4 +53,11 @@
             <state_interface name="velocity"/>
         </joint>
+        <joint name="${prefix}left_arm_joint_7">
+            <param name="node_id">27</param>
+            <param name="start_enabled">false</param>
+            <command_interface name="position"/>
+            <state_interface name="position"/>
+            <state_interface name="velocity"/>
+        </joint>
         <!-- Right Arm Joints -->
         <joint name="${prefix}right_arm_joint_1">
@@ -96,11 +103,4 @@
             <state_interface name="velocity"/>
         </joint>
-        <joint name="${prefix}right_arm_joint_7">
-            <param name="node_id">17</param>
-            <param name="start_enabled">false</param>
-            <command_interface name="position"/>
-            <state_interface name="position"/>
-            <state_interface name="velocity"/>
-        </joint>
     </ros2_control>
   </xacro:macro>

File: description/urdf/gripper_leader_supre_robot.urdf.xacro (robot description, xacro)
@@ -3,25 +3,17 @@
   <xacro:arg name="use_mock_hardware" default="false" />
   <xacro:arg name="prefix" default="" />
-  <xacro:arg name="param_can_device_index" default="1" />
+  <xacro:arg name="param_can_device_index" default="0" />
   <xacro:arg name="param_can_baud_rate" default="1000" />
   <xacro:arg name="param_device" default="/dev/ttyTHS1" />
   <xacro:arg name="param_baud_rate" default="115200" />
   <xacro:arg name="param_max_stroke" default="0.04" />
-  <xacro:include filename="$(find supre_robot_control)/urdf/supre_robot_description.urdf.xacro" />
+  <xacro:include filename="$(find supre_robot_control)/urdf/leader_supre_robot_description.urdf.xacro" />
   <!-- Import joints ros2_control description -->
-  <xacro:include filename="$(find supre_robot_control)/ros2_control/gripper_follower_joints.ros2_control.xacro" />
-  <!-- Import gripper description -->
-  <xacro:include filename="$(find supre_robot_control)/ros2_control/gripper.ros2_control.xacro" />
+  <xacro:include filename="$(find supre_robot_control)/ros2_control/gripper_leader_joints.ros2_control.xacro" />
   <link name="world"/>
   <xacro:create_robot prefix="$(arg prefix)">
   </xacro:create_robot>
-  <xacro:gripper_system
-    name="FollowerMisumiGripper" prefix="$(arg prefix)"
-    use_mock_hardware="$(arg use_mock_hardware)"
-    param_device="$(arg param_device)"
-    param_baud_rate="$(arg param_baud_rate)"
-    param_max_stroke="$(arg param_max_stroke)" />
   <xacro:joints_system
-    name="FollowerEyouSystem" prefix="$(arg prefix)"
+    name="LeaderEyouSystem" prefix="$(arg prefix)"
     use_mock_hardware="$(arg use_mock_hardware)"
     param_can_device_index="$(arg param_can_device_index)"
