Commit message: test

File: description/ros2_control/gripper_leader_joints.ros2_control.xacro (robot description, xacro)
@@ -103,4 +103,11 @@
             <state_interface name="velocity"/>
         </joint>
+        <joint name="${prefix}right_arm_joint_7">
+            <param name="node_id">17</param>
+            <param name="start_enabled">false</param>
+            <command_interface name="position"/>
+            <state_interface name="position"/>
+            <state_interface name="velocity"/>
+        </joint>
     </ros2_control>
   </xacro:macro>

File: description/urdf/gripper_follower_supre_robot.urdf.xacro (robot description, xacro)
@@ -6,4 +6,6 @@
   <xacro:arg name="param_can_baud_rate" default="1000" />
   <xacro:arg name="param_device" default="/dev/ttyTHS1" />
+  <xacro:arg name="param_device_left" default="/dev/ttyTHS1" />
+  <xacro:arg name="param_device_right" default="/dev/ttyTHS2" />
   <xacro:arg name="param_baud_rate" default="115200" />
   <xacro:arg name="param_max_stroke" default="0.04" />
@@ -12,14 +14,21 @@
   <xacro:include filename="$(find supre_robot_control)/ros2_control/gripper_follower_joints.ros2_control.xacro" />
   <!-- Import gripper description -->
-  <xacro:include filename="$(find supre_robot_control)/ros2_control/gripper.ros2_control.xacro" />
+  <xacro:include filename="$(find supre_robot_control)/ros2_control/gripper_left.ros2_control.xacro" />
+  <xacro:include filename="$(find supre_robot_control)/ros2_control/gripper_right.ros2_control.xacro" />
   <link name="world"/>
   <xacro:create_robot prefix="$(arg prefix)">
   </xacro:create_robot>
-  <xacro:gripper_system
-    name="FollowerMisumiGripper" prefix="$(arg prefix)"
+  <xacro:gripper_system_left
+    name="FollowerMisumiGripperLeft" prefix="$(arg prefix)"
     use_mock_hardware="$(arg use_mock_hardware)"
-    param_device="$(arg param_device)"
+    param_device="$(arg param_device_left)"
     param_baud_rate="$(arg param_baud_rate)"
     param_max_stroke="$(arg param_max_stroke)" />
+  <xacro:gripper_system_right
+    name="FollowerMisumiGripperRight" prefix="$(arg prefix)"
+    use_mock_hardware="$(arg use_mock_hardware)"
+    param_device="$(arg param_device_right)"
+    param_baud_rate="$(arg param_baud_rate)"
+    param_max_stroke="$(arg param_max_stroke)"/>
   <xacro:joints_system
     name="FollowerEyouSystem" prefix="$(arg prefix)"
